File: schema/connectors.sch (EAGLE design)
At the start: 26 parts, among them X1 ALARM, X2 22-23-2091

Commit message: Some I/O redefined
Parts:
- added LED1, LED2: LAP4-BOTTOM, led:LAP4-BOTTOM
- added R15, R17, R18, R19, R20: 10k, rcl:R-EU_0204/7
- added R16: 120, rcl:R-EU_0204/7
- added S1, S2, S3, S4, S5: TL32PO, switch:TL32PO
- R14: value 330 -> 120
Connections:
- net ELEMENT_A renamed WATER_HEATER_ELEMENT
- net FAN renamed FURNACE_FAN
- net HEATER renamed FURNACE_HEATER
- net TRANSPORT1 renamed FURNACE_TRANSPORT1
- net TRANSPORT2 renamed FURNACE_TRANSPORT2
- removed net ELEMENT_B: R9.1, SV1.36
- new net FORCE_TRANSPORT: R15.1, R16.1, S1.S
- new net FURNACEACTIVE: SV1.36
- new net FURNACE_ACTIVE: R9.1
- new net N$10: LED2.A, R14.1
- new net RED: SV1.15
- new net RETURN: R17.1, R18.1, R19.1, R20.1, S2.S, S3.S, S4.S, S5.S
- net +3V3: now also LED1.A, R14.2, R15.2, R17.2, R18.2, R19.2, R20.2
- net GND: now also LED2.C, S1.P, S2.P, S3.P, S4.P, S5.P
- net GREEN: no longer R14.1
- net N$3: now also LED1.C, R16.2; no longer R14.2, X2-7.S
Other:
- note added: "To Beijing"
- moved on the sheet: R14
